File: pcb.sch (KiCad schematic (older format))
At the start: 24 parts, among them SW1 SW_Push, U1 ATmega32U4-AU, Y1 16MHz

Commit message: update pcb with new components
Parts:
- removed D1, D2, D3, D4: D_Small, Diode_SMD:D_SOD-123, symbol Device:D_Small
- removed MX1, MX2, MX3, MX4: MX-NoLED, MX_Alps_Hybrid:MX-1.5U, symbol MX_Alps_Hybrid:MX-NoLED
- C7: footprint Diode_SMD:D_SOD-123 -> Capacitor_SMD:C_0805_2012Metric
- renumbered C4 to C1, C5 to C2, C6 to C3, C1 to C4, C2 to C5, C3 to C6, R3 to R1, R1 to R3
Changed lines of the file:
@@
 $EndComp
 $Comp
-L power:+5V #PWR0101
+L power:+5V #PWR02
 U 1 1 5E4B5E51
 P 5050 1350
-F 0 "#PWR0101" H 5050 1200 50  0001 C CNN
+F 0 "#PWR02" H 5050 1200 50  0001 C CNN
 F 1 "+5V" H 5065 1523 50  0000 C CNN
 F 2 "" H 5050 1350 50  0001 C CNN
@@
 Connection ~ 5050 1500
 $Comp
-L power:GND #PWR0102
+L power:GND #PWR013
 U 1 1 5E4B656C
 P 4700 5100
-F 0 "#PWR0102" H 4700 4850 50  0001 C CNN
+F 0 "#PWR013" H 4700 4850 50  0001 C CNN
 F 1 "GND" H 4705 4927 50  0000 C CNN
 F 2 "" H 4700 5100 50  0001 C CNN
@@
 $EndComp
 $Comp
-L power:GND #PWR0103
+L power:GND #PWR010
 U 1 1 5E4B795A
 P 6550 3900
-F 0 "#PWR0103" H 6550 3650 50  0001 C CNN
+F 0 "#PWR010" H 6550 3650 50  0001 C CNN
 F 1 "GND" H 6555 3727 50  0000 C CNN
 F 2 "" H 6550 3900 50  0001 C CNN
@@
 $EndComp
 $Comp
-L Device:R_Small R1
+L Device:R_Small R3
 U 1 1 5E4B86F1
 P 3900 2900
-F 0 "R1" V 3704 2900 50  0000 C CNN
+F 0 "R3" V 3704 2900 50  0000 C CNN
 F 1 "22" V 3795 2900 50  0000 C CNN
 F 2 "Resistor_SMD:R_0805_2012Metric" H 3900 2900 50  0001 C CNN
@@
 	3800 2900 3600 2900
 $Comp
-L Device:C_Small C6
+L Device:C_Small C3
 U 1 1 5E4B9734
 P 3700 3200
-F 0 "C6" H 3608 3154 50  0000 R CNN
+F 0 "C3" H 3608 3154 50  0000 R CNN
 F 1 "1uF" H 3608 3245 50  0000 R CNN
 F 2 "Capacitor_SMD:C_0805_2012Metric" H 3700 3200 50  0001 C CNN
@@
 $EndComp
 $Comp
-L power:GND #PWR0104
+L power:GND #PWR09
 U 1 1 5E4BA792
 P 3700 3550
-F 0 "#PWR0104" H 3700 3300 50  0001 C CNN
+F 0 "#PWR09" H 3700 3300 50  0001 C CNN
 F 1 "GND" H 3705 3377 50  0000 C CNN
 F 2 "" H 3700 3550 50  0001 C CNN
@@
 	3700 3300 3700 3550
 $Comp
-L Device:C_Small C1
+L Device:C_Small C4
 U 1 1 5E4BAFEB
 P 2800 4250
-F 0 "C1" H 2892 4296 50  0000 L CNN
+F 0 "C4" H 2892 4296 50  0000 L CNN
 F 1 "0.1uF" H 2892 4205 50  0000 L CNN
 F 2 "Capacitor_SMD:C_0805_2012Metric" H 2800 4250 50  0001 C CNN
@@
 $EndComp
 $Comp
-L Device:C_Small C2
+L Device:C_Small C5
 U 1 1 5E4BB424
 P 3200 4250
-F 0 "C2" H 3292 4296 50  0000 L CNN
+F 0 "C5" H 3292 4296 50  0000 L CNN
 F 1 "0.1uF" H 3292 4205 50  0000 L CNN
 F 2 "Capacitor_SMD:C_0805_2012Metric" H 3200 4250 50  0001 C CNN
@@
 $EndComp
 $Comp
-L Device:C_Small C3
+L Device:C_Small C6
 U 1 1 5E4BBA01
 P 3600 4250
-F 0 "C3" H 3692 4296 50  0000 L CNN
+F 0 "C6" H 3692 4296 50  0000 L CNN
 F 1 "0.1uF" H 3692 4205 50  0000 L CNN
 F 2 "Capacitor_SMD:C_0805_2012Metric" H 3600 4250 50  0001 C CNN
@@
 F 0 "C7" H 4092 4296 50  0000 L CNN
 F 1 "10uF" H 4092 4205 50  0000 L CNN
-F 2 "Diode_SMD:D_SOD-123" H 4000 4250 50  0001 C CNN
+F 2 "Capacitor_SMD:C_0805_2012Metric" H 4000 4250 50  0001 C CNN
 F 3 "~" H 4000 4250 50  0001 C CNN
 	1    4000 4250
@@
 	3600 4350 4000 4350
 $Comp
-L power:GND #PWR0105
+L power:GND #PWR012
 U 1 1 5E4BC986
 P 3400 4500
-F 0 "#PWR0105" H 3400 4250 50  0001 C CNN
+F 0 "#PWR012" H 3400 4250 50  0001 C CNN
 F 1 "GND" H 3405 4327 50  0000 C CNN
 F 2 "" H 3400 4500 50  0001 C CNN
@@
 $EndComp
 $Comp
-L power:+5V #PWR0106
+L power:+5V #PWR011
 U 1 1 5E4BCE01
 P 3400 4000
-F 0 "#PWR0106" H 3400 3850 50  0001 C CNN
+F 0 "#PWR011" H 3400 3850 50  0001 C CNN
 F 1 "+5V" H 3415 4173 50  0000 C CNN
 F 2 "" H 3400 4000 50  0001 C CNN
@@
 	3200 4350 3600 4350
 $Comp
-L power:+5V #PWR0107
+L power:+5V #PWR08
 U 1 1 5E4BF663
 P 4350 2600
-F 0 "#PWR0107" H 4350 2450 50  0001 C CNN
+F 0 "#PWR08" H 4350 2450 50  0001 C CNN
 F 1 "+5V" H 4365 2773 50  0000 C CNN
 F 2 "" H 4350 2600 50  0001 C CNN
@@
 	4100 2200 4550 2200
 $Comp
-L Device:C_Small C4
+L Device:C_Small C1
 U 1 1 5E4C524F
 P 3700 1900
-F 0 "C4" V 3471 1900 50  0000 C CNN
+F 0 "C1" V 3471 1900 50  0000 C CNN
 F 1 "22pF" V 3562 1900 50  0000 C CNN
 F 2 "Capacitor_SMD:C_0805_2012Metric" H 3700 1900 50  0001 C CNN
@@
 $EndComp
 $Comp
-L Device:C_Small C5
+L Device:C_Small C2
 U 1 1 5E4C5802
 P 3700 2300
-F 0 "C5" V 3471 2300 50  0000 C CNN
+F 0 "C2" V 3471 2300 50  0000 C CNN
 F 1 "22pF" V 3562 2300 50  0000 C CNN
 F 2 "Capacitor_SMD:C_0805_2012Metric" H 3700 2300 50  0001 C CNN
@@
 	3600 1900 3600 2300
 $Comp
-L power:GND #PWR0108
+L power:GND #PWR07
 U 1 1 5E4C8419
 P 3600 2400
-F 0 "#PWR0108" H 3600 2150 50  0001 C CNN
+F 0 "#PWR07" H 3600 2150 50  0001 C CNN
 F 1 "GND" H 3605 2227 50  0000 C CNN
 F 2 "" H 3600 2400 50  0001 C CNN
@@
 	4550 1800 4500 1800
 $Comp
-L power:GND #PWR0109
+L power:GND #PWR05
 U 1 1 5E4CB2FF
 P 3950 1750
-F 0 "#PWR0109" H 3950 1500 50  0001 C CNN
+F 0 "#PWR05" H 3950 1500 50  0001 C CNN
 F 1 "GND" H 3955 1577 50  0000 C CNN
 F 2 "" H 3950 1750 50  0001 C CNN
@@
 	4050 1750 4050 1800
 $Comp
-L Device:R_Small R3
+L Device:R_Small R1
 U 1 1 5E4CC718
 P 4500 1500
-F 0 "R3" H 4559 1546 50  0000 L CNN
+F 0 "R1" H 4559 1546 50  0000 L CNN
 F 1 "10k" H 4559 1455 50  0000 L CNN
 F 2 "Resistor_SMD:R_0805_2012Metric" H 4500 1500 50  0001 C CNN
@@
 	4500 1800 4450 1800
 $Comp
-L power:+5V #PWR0110
+L power:+5V #PWR01
 U 1 1 5E4CD753
 P 4500 1300
-F 0 "#PWR0110" H 4500 1150 50  0001 C CNN
+F 0 "#PWR01" H 4500 1150 50  0001 C CNN
 F 1 "+5V" H 4515 1473 50  0000 C CNN
 F 2 "" H 4500 1300 50  0001 C CNN
@@
 	7150 1650 7400 1650
 $Comp
-L power:VCC #PWR0111
+L power:VCC #PWR03
 U 1 1 5E4D65C7
 P 7400 1650
-F 0 "#PWR0111" H 7400 1500 50  0001 C CNN
+F 0 "#PWR03" H 7400 1500 50  0001 C CNN
 F 1 "VCC" H 7417 1823 50  0000 C CNN
 F 2 "" H 7400 1650 50  0001 C CNN
@@
 	7400 1650 7750 1650
 $Comp
-L power:+5V #PWR0112
+L power:+5V #PWR04
 U 1 1 5E4D6B03
 P 8300 1650
-F 0 "#PWR0112" H 8300 1500 50  0001 C CNN
+F 0 "#PWR04" H 8300 1500 50  0001 C CNN
 F 1 "+5V" H 8315 1823 50  0000 C CNN
 F 2 "" H 8300 1650 50  0001 C CNN
@@
 D+
 $Comp
-L power:GND #PWR0113
+L power:GND #PWR06
 U 1 1 5E4D8A33
 P 7250 2050
-F 0 "#PWR0113" H 7250 1800 50  0001 C CNN
+F 0 "#PWR06" H 7250 1800 50  0001 C CNN
 F 1 "GND" H 7255 1877 50  0000 C CNN
 F 2 "" H 7250 2050 50  0001 C CNN
@@
 Wire Wire Line
 	7250 2050 7150 2050
-$Comp
-L MX_Alps_Hybrid:MX-NoLED MX1
-U 1 1 5E4D9DFD
-P 1850 1600
-F 0 "MX1" H 1883 1823 60  0000 C CNN
-F 1 "MX-NoLED" H 1883 1749 20  0000 C CNN
-F 2 "MX_Alps_Hybrid:MX-1.5U" H 1225 1575 60  0001 C CNN
-F 3 "" H 1225 1575 60  0001 C CNN
-	1    1850 1600
-	1    0    0    -1
-$EndComp
-$Comp
-L Device:D_Small D1
-U 1 1 5E4DA8FB
-P 1600 1850
-F 0 "D1" V 1646 1782 50  0000 R CNN
-F 1 "D_Small" V 1555 1782 50  0000 R CNN
-F 2 "Diode_SMD:D_SOD-123" V 1600 1850 50  0001 C CNN
-F 3 "~" V 1600 1850 50  0001 C CNN
-	1    1600 1850
-	0    -1   -1   0
-$EndComp
-Wire Wire Line
-	1600 1750 1800 1750
-$Comp
-L MX_Alps_Hybrid:MX-NoLED MX3
-U 1 1 5E4E28C8
-P 2550 1600
-F 0 "MX3" H 2583 1823 60  0000 C CNN
-F 1 "MX-NoLED" H 2583 1749 20  0000 C CNN
-F 2 "MX_Alps_Hybrid:MX-1.5U" H 1925 1575 60  0001 C CNN
-F 3 "" H 1925 1575 60  0001 C CNN
-	1    2550 1600
-	1    0    0    -1
-$EndComp
-$Comp
-L Device:D_Small D3
-U 1 1 5E4E28CE
-P 2300 1850
-F 0 "D3" V 2346 1782 50  0000 R CNN
-F 1 "D_Small" V 2255 1782 50  0000 R CNN
-F 2 "Diode_SMD:D_SOD-123" V 2300 1850 50  0001 C CNN
-F 3 "~" V 2300 1850 50  0001 C CNN
-	1    2300 1850
-	0    -1   -1   0
-$EndComp
-Wire Wire Line
-	2300 1750 2500 1750
-$Comp
-L MX_Alps_Hybrid:MX-NoLED MX4
-U 1 1 5E4E35DD
-P 2600 2350
-F 0 "MX4" H 2633 2573 60  0000 C CNN
-F 1 "MX-NoLED" H 2633 2499 20  0000 C CNN
-F 2 "MX_Alps_Hybrid:MX-1.5U" H 1975 2325 60  0001 C CNN
-F 3 "" H 1975 2325 60  0001 C CNN
-	1    2600 2350
-	1    0    0    -1
-$EndComp
-$Comp
-L Device:D_Small D4
-U 1 1 5E4E35E3
-P 2350 2600
-F 0 "D4" V 2396 2532 50  0000 R CNN
-F 1 "D_Small" V 2305 2532 50  0000 R CNN
-F 2 "Diode_SMD:D_SOD-123" V 2350 2600 50  0001 C CNN
-F 3 "~" V 2350 2600 50  0001 C CNN
-	1    2350 2600
-	0    -1   -1   0
-$EndComp
-Wire Wire Line
-	2350 2500 2550 2500
-$Comp
-L MX_Alps_Hybrid:MX-NoLED MX2
-U 1 1 5E4E4730
-P 1850 2350
-F 0 "MX2" H 1883 2573 60  0000 C CNN
-F 1 "MX-NoLED" H 1883 2499 20  0000 C CNN
-F 2 "MX_Alps_Hybrid:MX-1.5U" H 1225 2325 60  0001 C CNN
-F 3 "" H 1225 2325 60  0001 C CNN
-	1    1850 2350
-	1    0    0    -1
-$EndComp
-$Comp
-L Device:D_Small D2
-U 1 1 5E4E4736
-P 1600 2600
-F 0 "D2" V 1646 2532 50  0000 R CNN
-F 1 "D_Small" V 1555 2532 50  0000 R CNN
-F 2 "Diode_SMD:D_SOD-123" V 1600 2600 50  0001 C CNN
-F 3 "~" V 1600 2600 50  0001 C CNN
-	1    1600 2600
-	0    -1   -1   0
-$EndComp
-Wire Wire Line
-	1600 2500 1800 2500
-Wire Wire Line
-	2000 2300 2000 1550
-Connection ~ 2000 1550
-Wire Wire Line
-	2000 1550 2000 1250
-Wire Wire Line
-	2750 2300 2750 1250
-Wire Wire Line
-	2300 1950 1600 1950
-Connection ~ 1600 1950
-Wire Wire Line
-	1600 1950 1450 1950
-Wire Wire Line
-	2350 2700 1600 2700
-Connection ~ 1600 2700
-Wire Wire Line
-	1600 2700 1450 2700
-Text GLabel 2000 1250 1    50   Input ~ 0
-COL0
-Text GLabel 2750 1250 1    50   Input ~ 0
-COL1
-Text GLabel 1450 1950 0    50   Input ~ 0
-ROW0
-Text GLabel 1450 2700 0    50   Input ~ 0
-ROW1
 $EndSCHEMATC

Commit message: finish wiring pcb
Parts:
- added D1, D2, D3, D4: SOD-123, Diode_SMD:D_SOD-123, symbol Device:D_Small
- added MX1, MX2, MX3, MX4: MX-1U, MX_Alps_Hybrid:MX-1U, symbol MX_Alps_Hybrid:MX-NoLED
Connections:
- new net: D1.2 (A), MX1.2 (ROW)
- new net: D2.2 (A), MX2.2 (ROW)
- new net: D3.2 (A), MX3.2 (ROW)
- new net: D4.2 (A), MX4.2 (ROW)
- new net COL0: MX1.1 (COL), MX3.1 (COL)
- new net COL1: MX2.1 (COL), MX4.1 (COL)
- new net ROW0: D1.1 (K), D2.1 (K)
- new net ROW1: D3.1 (K), D4.1 (K)
Changed lines of the file:
@@
 $EndDescr
-$Comp
-L MCU_Microchip_ATmega:ATmega32U4-AU U1
-U 1 1 5E4B48A7
-P 5150 3300
-F 0 "U1" H 5150 1411 50  0000 C CNN
-F 1 "ATmega32U4-AU" H 5150 1320 50  0000 C CNN
-F 2 "Package_QFP:TQFP-44_10x10mm_P0.8mm" H 5150 3300 50  0001 C CIN
-F 3 "http://ww1.microchip.com/downloads/en/DeviceDoc/Atmel-7766-8-bit-AVR-ATmega16U4-32U4_Datasheet.pdf" H 5150 3300 50  0001 C CNN
-	1    5150 3300
-	1    0    0    -1
-$EndComp
 $Comp
 L power:+5V #PWR02
@@
 $EndComp
 Wire Wire Line
-	5750 3900 6100 3900
-Wire Wire Line
 	6300 3900 6550 3900
 $Comp
@@
 Wire Wire Line
 	7250 2050 7150 2050
+$Comp
+L MX_Alps_Hybrid:MX-NoLED MX1
+U 1 1 5E565D2D
+P 7950 3450
+F 0 "MX1" H 7983 3673 60  0000 C CNN
+F 1 "MX-1U" H 7983 3599 20  0000 C CNN
+F 2 "MX_Alps_Hybrid:MX-1U" H 7325 3425 60  0001 C CNN
+F 3 "" H 7325 3425 60  0001 C CNN
+	1    7950 3450
+	1    0    0    -1
+$EndComp
+Wire Wire Line
+	7900 3600 7800 3600
+$Comp
+L Device:D_Small D1
+U 1 1 5E5667F0
+P 7800 3700
+F 0 "D1" H 7846 3791 50  0000 R BNN
+F 1 "SOD-123" H 7873 3791 50  0000 L BNN
+F 2 "Diode_SMD:D_SOD-123" V 7800 3700 50  0001 C CNN
+F 3 "~" V 7800 3700 50  0001 C CNN
+	1    7800 3700
+	0    -1   -1   0
+$EndComp
+$Comp
+L MX_Alps_Hybrid:MX-NoLED MX2
+U 1 1 5E56DDF8
+P 8700 3450
+F 0 "MX2" H 8733 3673 60  0000 C CNN
+F 1 "MX-1U" H 8733 3599 20  0000 C CNN
+F 2 "MX_Alps_Hybrid:MX-1U" H 8075 3425 60  0001 C CNN
+F 3 "" H 8075 3425 60  0001 C CNN
+	1    8700 3450
+	1    0    0    -1
+$EndComp
+Wire Wire Line
+	8650 3600 8550 3600
+$Comp
+L Device:D_Small D2
+U 1 1 5E56DDFF
+P 8550 3700
+F 0 "D2" H 8596 3791 50  0000 R BNN
+F 1 "SOD-123" H 8623 3791 50  0000 L BNN
+F 2 "Diode_SMD:D_SOD-123" V 8550 3700 50  0001 C CNN
+F 3 "~" V 8550 3700 50  0001 C CNN
+	1    8550 3700
+	0    -1   -1   0
+$EndComp
+$Comp
+L MX_Alps_Hybrid:MX-NoLED MX3
+U 1 1 5E56F275
+P 7950 4200
+F 0 "MX3" H 7983 4423 60  0000 C CNN
+F 1 "MX-1U" H 7983 4349 20  0000 C CNN
+F 2 "MX_Alps_Hybrid:MX-1U" H 7325 4175 60  0001 C CNN
+F 3 "" H 7325 4175 60  0001 C CNN
+	1    7950 4200
+	1    0    0    -1
+$EndComp
+Wire Wire Line
+	7900 4350 7800 4350
+$Comp
+L Device:D_Small D3
+U 1 1 5E56F27C
+P 7800 4450
+F 0 "D3" H 7846 4541 50  0000 R BNN
+F 1 "SOD-123" H 7873 4541 50  0000 L BNN
+F 2 "Diode_SMD:D_SOD-123" V 7800 4450 50  0001 C CNN
+F 3 "~" V 7800 4450 50  0001 C CNN
+	1    7800 4450
+	0    -1   -1   0
+$EndComp
+$Comp
+L MX_Alps_Hybrid:MX-NoLED MX4
+U 1 1 5E5716AE
+P 8700 4200
+F 0 "MX4" H 8733 4423 60  0000 C CNN
+F 1 "MX-1U" H 8733 4349 20  0000 C CNN
+F 2 "MX_Alps_Hybrid:MX-1U" H 8075 4175 60  0001 C CNN
+F 3 "" H 8075 4175 60  0001 C CNN
+	1    8700 4200
+	1    0    0    -1
+$EndComp
+Wire Wire Line
+	8650 4350 8550 4350
+$Comp
+L Device:D_Small D4
+U 1 1 5E5716B5
+P 8550 4450
+F 0 "D4" H 8596 4541 50  0000 R BNN
+F 1 "SOD-123" H 8623 4541 50  0000 L BNN
+F 2 "Diode_SMD:D_SOD-123" V 8550 4450 50  0001 C CNN
+F 3 "~" V 8550 4450 50  0001 C CNN
+	1    8550 4450
+	0    -1   -1   0
+$EndComp
+Wire Wire Line
+	8100 3100 8100 3400
+Connection ~ 8100 3400
+Wire Wire Line
+	8100 3400 8100 4150
+Wire Wire Line
+	8850 3100 8850 3400
+Connection ~ 8850 3400
+Wire Wire Line
+	8850 3400 8850 4150
+Wire Wire Line
+	8550 3800 7800 3800
+Connection ~ 7800 3800
+Wire Wire Line
+	7800 3800 7500 3800
+Wire Wire Line
+	8550 4550 7800 4550
+Connection ~ 7800 4550
+Wire Wire Line
+	7800 4550 7500 4550
+Text GLabel 7500 4550 0    50   Input ~ 0
+ROW1
+Text GLabel 7500 3800 0    50   Input ~ 0
+ROW0
+Text GLabel 8100 3100 1    50   Input ~ 0
+COL0
+Text GLabel 8850 3100 1    50   Input ~ 0
+COL1
+Text GLabel 5950 2300 0    50   Output ~ 0
+COL0
+Wire Wire Line
+	5750 3900 6100 3900
+$Comp
+L MCU_Microchip_ATmega:ATmega32U4-AU U1
+U 1 1 5E4B48A7
+P 5150 3300
+F 0 "U1" H 5150 1411 50  0000 C CNN
+F 1 "ATmega32U4-AU" H 5150 1320 50  0000 C CNN
+F 2 "Package_QFP:TQFP-44_10x10mm_P0.8mm" H 5150 3300 50  0001 C CIN
+F 3 "http://ww1.microchip.com/downloads/en/DeviceDoc/Atmel-7766-8-bit-AVR-ATmega16U4-32U4_Datasheet.pdf" H 5150 3300 50  0001 C CNN
+	1    5150 3300
+	1    0    0    -1
+$EndComp
 $EndSCHEMATC
